File: AeroAngleSense/_autosave-AeroAngleSense.kicad_pcb (KiCad board)
At the start: 2 copper layers, 15 x 55 mm, 23 parts, among them IC1 STM32F042F6P6, IC2 TMP127EDBVRQ1, IC3 TPS62842DGRR, J1 SM06B-GHS-TBT, J7 SM04B-GHS-TBT

Commit message: 배선 작업_1
Routing:
- net GND: track 26.0 -> 33.0 mm, vias 11 -> 12
- net +3.3V: track 13.3 -> 18.7 mm
- net +5V: track 0.00 -> 4.49 mm
- net /TMP_MISO: track 0.00 -> 2.32 mm
Changed lines of the file:
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@@
+	)
+	(segment
+		(start 31.051 44.349)
+		(end 29.126 44.349)
+		(width 0.2)
+		(layer "F.Cu")
+		(net 1)
 	)
 	(segment
@@
 	)
 	(segment
+		(start 27.925 58.15)
+		(end 27.675 58.4)
+		(width 0.4)
+		(layer "F.Cu")
+		(net 1)
+	)
+	(segment
+		(start 28.7 44.775)
+		(end 28.7 46)
+		(width 0.2)
+		(layer "F.Cu")
+		(net 1)
+	)
+	(segment
+		(start 29.75 58.15)
+		(end 27.925 58.15)
+		(width 0.4)
+		(layer "F.Cu")
+		(net 1)
+	)
+	(segment
 		(start 25.275 56.375)
 		(end 25.875 56.375)
@@
 	)
 	(segment
+		(start 31.4 45.25)
+		(end 31.4 44.698)
+		(width 0.2)
+		(layer "F.Cu")
+		(net 1)
+	)
+	(segment
 		(start 24.825 56.825)
 		(end 25.275 56.375)
@@
 	)
 	(segment
+		(start 29.126 44.349)
+		(end 28.7 44.775)
+		(width 0.2)
+		(layer "F.Cu")
+		(net 1)
+	)
+	(segment
 		(start 24.825 62.125)
 		(end 25.375 62.125)
@@
 	)
 	(segment
+		(start 31.4 44.698)
+		(end 31.051 44.349)
+		(width 0.2)
+		(layer "F.Cu")
+		(net 1)
+	)
+	(segment
 		(start 30 36.6)
 		(end 30 37.5)
@@
 	)
 	(via
+		(at 28.7 46)
+		(size 0.4)
+		(drill 0.3)
+		(layers "F.Cu" "B.Cu")
+		(net 1)
+	)
+	(via
 		(at 31.5 39)
 		(size 0.4)
@@
 	)
 	(segment
+		(start 30.45 42.75)
+		(end 29.175 42.75)
+		(width 0.2)
+		(layer "F.Cu")
+		(net 2)
+	)
+	(segment
 		(start 24.525 50.75)
 		(end 24.525 52.25)
@@
 	)
 	(segment
+		(start 29.175 42.75)
+		(end 28.7 43.225)
+		(width 0.2)
+		(layer "F.Cu")
+		(net 2)
+	)
+	(segment
 		(start 24.075 48.935)
 		(end 24.075 50.3)
@@
 	)
 	(segment
+		(start 24.075 41.45)
+		(end 24.275 41.25)
+		(width 0.2)
+		(layer "F.Cu")
+		(net 2)
+	)
+	(segment
 		(start 21.75 58.4)
 		(end 21.25 57.9)
@@
 	)
 	(segment
+		(start 24.075 43.065)
+		(end 24.075 41.45)
+		(width 0.2)
+		(layer "F.Cu")
+		(net 2)
+	)
+	(segment
 		(start 23.725 56.375)
 		(end 23.725 57.95)
@@
 	)
 	(segment
+		(start 24.275 39.75)
+		(end 24.275 41.25)
+		(width 0.2)
+		(layer "F.Cu")
+		(net 2)
+	)
+	(segment
 		(start 23.725 57.95)
 		(end 23.275 58.4)
@@
 	)
 	(segment
+		(start 29.75 59.7)
+		(end 29.574 59.876)
+		(width 0.4)
+		(layer "F.Cu")
+		(net 4)
+	)
+	(segment
+		(start 29.574 59.876)
+		(end 27.675 59.876)
+		(width 0.4)
+		(layer "F.Cu")
+		(net 4)
+	)
+	(segment
+		(start 29.75 59.7)
+		(end 29.1 60.35)
+		(width 0.4)
+		(layer "F.Cu")
+		(net 4)
+	)
+	(segment
+		(start 29.1 60.35)
+		(end 27.675 60.35)
+		(width 0.4)
+		(layer "F.Cu")
+		(net 4)
+	)
+	(segment
 		(start 27.5 38.325)
 		(end 28.675 39.5)
@@
 	)
 	(segment
-		(start 23.275 62.025)
-		(end 23.175 62.125)
-		(width 0.2)
-		(layer "F.Cu")
-		(net 24)
-	)
-	(segment
+		(start 32.35 45.25)
+		(end 32.914064 45.25)
+		(width 0.2)
+		(layer "F.Cu")
+		(net 8)
+	)
+	(segment
+		(start 33.95 44.214064)
+		(end 33.95 43.925)
+		(width 0.2)
+		(layer "F.Cu")
+		(net 8)
+	)
+	(segment
+		(start 32.914064 45.25)
+		(end 33.95 44.214064)
+		(width 0.2)
+		(layer "F.Cu")
+		(net 8)
+	)
+	(segment
