File: AeroAngleSense/AeroAngleSense.kicad_pcb (KiCad board)
At the start: 2 copper layers, 15 x 55 mm, 23 parts, among them IC1 STM32F042F6P6, IC2 TMP127EDBVRQ1, IC3 TPS62842DGRR, J1 SM06B-GHS-TBT, J7 SM04B-GHS-TBT

Commit message: 배선_2
Routing:
- net /I2C_SDA: track 0.00 -> 23.9 mm
- net /I2C_SCL: track 0.00 -> 22.7 mm
- net /POT_SEN: track 1.52 -> 18.4 mm, vias 0 -> 2
- net /USART2_TX: track 0.00 -> 15.9 mm, vias 0 -> 1
- net /TMP_MISO: track 0.00 -> 15.7 mm
- net /NRST: track 0.00 -> 15.7 mm, vias 0 -> 1
- net /TMP_MOSI: track 0.00 -> 13.7 mm
- net /SWDIO: track 0.00 -> 12.6 mm
- net GND: track 26.0 -> 38.7 mm, vias 11 -> 15
- net /TMP_CS: track 0.00 -> 12.1 mm
- net /SWCLK: track 0.00 -> 9.84 mm
- net +3.3V: track 13.3 -> 21.8 mm, vias 2 -> 4
- net +5V: track 0.00 -> 4.49 mm
- net Net-(IC1-PB8-BOOT0): track 0.00 -> 1.77 mm

Commit message: 배선_3
Parts:
- moved C7 0.32 mm to (30.1, 58.9)
- moved C8 0.32 mm to (24.8, 56.4)
- moved IC3 0.32 mm to (25.8, 59.4)
- moved L1 0.32 mm to (21.6, 58.6)
- moved R3 0.32 mm to (24.3, 62.1)
Routing:
- net /TMP_SCLK: track 0.00 -> 52.1 mm, vias 0 -> 2
- net +3.3V: track 21.8 -> 62.6 mm
- net +5V: track 4.49 -> 17.4 mm, vias 0 -> 2
- net GND: track 38.7 -> 39.1 mm, vias 15 -> 18

Commit message: 배선 최종
Routing:
- net GND: track 39.1 -> 55.5 mm, vias 18 -> 20
- net /I2C_SDA: track 24.2 -> 23.4 mm, vias 0 -> 2
Changed lines of the file:
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@@
 		(tags "capacitor")
 		(property "Reference" "C9"
-			(at 0 -1.43 90)
+			(at -0.2 8.1 90)
 			(layer "F.SilkS")
 			(effects
@@
 		(tags "mountinghole M2")
 		(property "Reference" "H2"
-			(at 0 -3.15 0)
+			(at -0.75 -3.8 0)
 			(layer "F.SilkS")
 			(effects
@@
 		(tags "Integrated Circuit")
 		(property "Reference" "IC2"
-			(at 0 0 90)
+			(at 2.4 2.6 90)
 			(layer "F.SilkS")
 			(effects
@@
 		(tags "connector jst GH SMT side horizontal entry 1.25mm pitch")
 		(property "Reference" "J7"
-			(at -0.225 -2.85 0)
+			(at -0.225 0.7 0)
 			(layer "F.SilkS")
 			(effects
@@
 		(at 21.575 58.575 90)
 		(property "Reference" "L1"
-			(at 0 -1.5 90)
+			(at -0.025 -2.575 90)
 			(unlocked yes)
 			(layer "F.SilkS")
@@
 		(tags "capacitor")
 		(property "Reference" "C5"
-			(at 0 -1.43 0)
+			(at -2.65 0.05 0)
 			(layer "F.SilkS")
 			(effects
@@
 		(tags "capacitor")
 		(property "Reference" "C6"
-			(at 0 -1.43 0)
+			(at -2.25 -0.05 0)
 			(layer "F.SilkS")
 			(effects
@@
 		(tags "resistor")
 		(property "Reference" "R2"
-			(at 0 -1.43 0)
+			(at 2.3 0.1 0)
 			(layer "F.SilkS")
 			(effects
@@
 		(tags "capacitor")
 		(property "Reference" "C3"
-			(at -1.775 0.5 0)
+			(at -2.3 0 0)
 			(layer "F.SilkS")
 			(effects
@@
 		(tags "capacitor")
 		(property "Reference" "C8"
-			(at 0 -1.43 0)
+			(at 1.175 -1.175 0)
 			(layer "F.SilkS")
 			(effects
@@
 		(tags "Through hole pin header THT 1x06 2.54mm single row")
 		(property "Reference" "J1"
-			(at 0 -2.38 0)
+			(at 0 -2.45 0)
 			(layer "F.SilkS")
 			(effects
@@
 		(tags "resistor")
 		(property "Reference" "R1"
-			(at 0 -1.43 90)
+			(at 0 1.15 270)
 			(layer "F.SilkS")
 			(effects
@@
 		(tags "mountinghole M2")
 		(property "Reference" "H3"
-			(at 0 -3.15 0)
+			(at 0.35 -3.8 0)
 			(layer "F.SilkS")
 			(effects
@@
 		(tags "Integrated Circuit")
 		(property "Reference" "IC3"
-			(at 0 0 0)
+			(at -7.4 1.025 0)
 			(layer "F.SilkS")
 			(effects
@@
 		(tags "mountinghole M2")
 		(property "Reference" "H4"
-			(at 0 -3.15 0)
+			(at 3.75 0 0)
 			(layer "F.SilkS")
 			(effects
@@
 		(tags "Hardware")
 		(property "Reference" "H1"
-			(at 0 0.27 0)
+			(at 10.5 -0.58 0)
 			(layer "F.SilkS")
 			(effects
@@
 	)
 	(segment
+		(start 28.7 46)
+		(end 28.699 46.001)
+		(width 0.2)
+		(layer "F.Cu")
+		(net 1)
+	)
+	(segment
 		(start 33.2 48.45)
 		(end 30.55 48.45)
@@
 	)
 	(segment
-		(start 23.425 50.3)
-		(end 23.425 48.935)
+		(start 31.4 46.2)
+		(end 31.2 46.4)
 		(width 0.2)
 		(layer "F.Cu")
@@
 	)
 	(segment
-		(start 31.051 44.349)
-		(end 29.126 44.349)
+		(start 22.024 66.301)
+		(end 21.099 65.376)
 		(width 0.2)
 		(layer "F.Cu")
@@
 	)
 	(segment
-		(start 23.425 50.3)
-		(end 22.975 50.75)
-		(width 0.2)
-		(layer "F.Cu")
-		(net 1)
-	)
-	(segment
 		(start 22.723 59.7)
 		(end 21.35 61.073)
@@
 	)
 	(segment
+		(start 26.575 65.425)
+		(end 25.699 66.301)
+		(width 0.2)
+		(layer "F.Cu")
+		(net 1)
+	)
+	(segment
+		(start 31.4 44.45)
+		(end 31.299 44.349)
+		(width 0.2)
+		(layer "F.Cu")
+		(net 1)
+	)
+	(segment
+		(start 26.575 64.9)
+		(end 26.575 65.425)
+		(width 0.2)
+		(layer "F.Cu")
+		(net 1)
+	)
+	(segment
+		(start 29.4 48.2)
+		(end 29.4 49.6)
+		(width 0.2)
+		(layer "F.Cu")
+		(net 1)
+	)
+	(segment
 		(start 22.725 41.25)
 		(end 21.65 41.25)
@@
 	(segment
 		(start 31.4 45.25)
-		(end 31.4 44.698)
+		(end 31.4 44.45)
 		(width 0.2)
 		(layer "F.Cu")
@@
 	)
 	(segment
-		(start 29.126 44.349)
-		(end 28.7 44.775)
-		(width 0.2)
-		(layer "F.Cu")
-		(net 1)
-	)
-	(segment
-		(start 27.1 64.9)
-		(end 27.8 64.2)
+		(start 23.425 48.935)
+		(end 23.425 50.3)
 		(width 0.2)
 		(layer "F.Cu")
@@
 	)
 	(segment
-		(start 31.4 44.698)
-		(end 31.051 44.349)
-		(width 0.2)
-		(layer "F.Cu")
-		(net 1)
-	)
-	(segment
-		(start 28.7 44.775)
-		(end 29.375 44.775)
+		(start 30 36.6)
+		(end 30 37.5)
 		(width 0.2)
 		(layer "F.Cu")
@@
 	)
 	(segment
-		(start 30 36.6)
-		(end 30 37.5)
+		(start 31.299 44.349)
+		(end 29.126 44.349)
 		(width 0.2)
 		(layer "F.Cu")
@@
 	)
 	(segment
-		(start 26.575 64.9)
-		(end 27.1 64.9)
-		(width 0.2)
-		(layer "F.Cu")
-		(net 1)
-	)
-	(segment
 		(start 25.8 60.225)
 		(end 27.075 61.5)
@@
 	)
 	(segment
+		(start 21.099 61.501)
+		(end 21.35 61.25)
+		(width 0.2)
+		(layer "F.Cu")
+		(net 1)
+	)
+	(segment
+		(start 29.4 49.6)
+		(end 28.418554 50.581446)
+		(width 0.2)
+		(layer "F.Cu")
+		(net 1)
+	)
+	(segment
+		(start 31.4 45.25)
+		(end 31.4 46.2)
+		(width 0.2)
+		(layer "F.Cu")
+		(net 1)
+	)
+	(segment
 		(start 22.975 50.75)
 		(end 22.975 52.25)
@@
 	)
 	(segment
-		(start 29.375 44.775)
-		(end 29.6 45)
+		(start 23.425 50.3)
+		(end 22.975 50.75)
+		(width 0.2)
+		(layer "F.Cu")
+		(net 1)
+	)
+	(segment
+		(start 21.099 65.376)
+		(end 21.099 61.501)
+		(width 0.2)
+		(layer "F.Cu")
+		(net 1)
+	)
+	(segment
+		(start 25.699 66.301)
+		(end 22.024 66.301)
 		(width 0.2)
 		(layer "F.Cu")
@@
 	)
 	(segment
+		(start 29.126 44.349)
+		(end 28.7 44.775)
+		(width 0.2)
+		(layer "F.Cu")
+		(net 1)
+	)
+	(segment
 		(start 26.006664 39.675)
 		(end 25.831665 39.500001)
@@
 		(net 1)
 	)
+	(segment
+		(start 28.7 44.775)
+		(end 28.7 46)
+		(width 0.2)
+		(layer "F.Cu")
+		(net 1)
+	)
 	(via
 		(at 30.4 48.6)
@@
 	)
 	(via
-		(at 27.8 64.2)
-		(size 0.4)
-		(drill 0.3)
-		(layers "F.Cu" "B.Cu")
-		(net 1)
-	)
-	(via
-		(at 29.6 45)
+		(at 29.4 48.2)
 		(size 0.4)
 		(drill 0.3)
@@
 	)
 	(via
+		(at 31.2 46.4)
+		(size 0.4)
+		(drill 0.3)
+		(layers "F.Cu" "B.Cu")
+		(net 1)
+	)
+	(via
 		(at 21.35 61.25)
 		(size 0.4)
@@
 	)
 	(via
+		(at 28.699 46.001)
+		(size 0.4)
+		(drill 0.3)
+		(layers "F.Cu" "B.Cu")
+		(net 1)
+	)
+	(via
 		(at 27.075 61.5)
 		(size 0.4)
@@
 		(net 1)
 	)
+	(via
+		(at 28.418554 50.581446)
+		(size 0.4)
+		(drill 0.3)
+		(layers "F.Cu" "B.Cu")
+		(net 1)
+	)
+	(segment
+		(start 28.699 46.001)
+		(end 28.699 47.499)
+		(width 0.2)
+		(layer "B.Cu")
+		(net 1)
+	)
+	(segment
+		(start 28.699 47.499)
+		(end 29.4 48.2)
+		(width 0.2)
+		(layer "B.Cu")
+		(net 1)
+	)
 	(segment
 		(start 32.834108 61.15)
@@
 	)
 	(segment
+		(start 25.425 64.8)
+		(end 25.325 64.9)
+		(width 0.2)
+		(layer "F.Cu")
+		(net 22)
+	)
+	(segment
 		(start 31.452 61.825)
-		(end 27.176 66.101)
+		(end 30.775 61.825)
+		(width 0.2)
+		(layer "F.Cu")
+		(net 22)
+	)
+	(segment
+		(start 30.775 61.825)
+		(end 27.8 64.8)
 		(width 0.2)
 		(layer "F.Cu")
@@
 	)
 	(segment
-		(start 25.926 66.101)
-		(end 25.325 65.5)
+		(start 25.874998 64.8)
+		(end 25.425 64.8)
 		(width 0.2)
 		(layer "F.Cu")
 		(net 22)
 	)
+	(via
+		(at 27.8 64.8)
+		(size 0.4)
+		(drill 0.3)
+		(layers "F.Cu" "B.Cu")
+		(net 22)
+	)
+	(via
+		(at 25.874998 64.8)
+		(size 0.4)
+		(drill 0.3)
+		(layers "F.Cu" "B.Cu")
+		(net 22)
+	)
 	(segment
-		(start 27.176 66.101)
-		(end 25.926 66.101)
+		(start 27.8 64.8)
+		(end 25.874998 64.8)
 		(width 0.2)
-		(layer "F.Cu")
+		(layer "B.Cu")
 		(net 22)
 	)

Commit message: 배선_4
Routing:
- net +3.3V: track 62.6 -> 59.9 mm
- net /USART2_TX: track 15.9 -> 17.2 mm
- net /NRST: track 15.7 -> 16.5 mm
- net /I2C_SDA: track 23.4 -> 23.3 mm, vias 2 -> 0
- net GND: vias 20 -> 19

Commit message: fix : route
Parts:
- renumbered J7 to J2, R4 to R3, R3 to R4, IC1 to U1, IC3 to U2, IC2 to U3
Routing:
- net GND: track 55.5 -> 15.4 mm, vias 19 -> 26
- net /TMP_SCLK: track 52.1 -> 16.0 mm
- net /I2C_SCL: track 23.5 -> 16.9 mm, vias 0 -> 2
- net /I2C_SDA: track 23.3 -> 17.3 mm, vias 0 -> 2
- net +5V: track 17.4 -> 11.6 mm, vias 2 -> 0
- net +3.3V: track 59.9 -> 56.5 mm, vias 4 -> 5
- net /POT_SEN: track 18.4 -> 16.5 mm
- net /NRST: track 16.5 -> 15.0 mm
- net /USART2_TX: track 17.2 -> 16.2 mm
- net /SWCLK: track 9.84 -> 10.8 mm
- net /TMP_MISO: track 15.7 -> 16.2 mm
- added copper zone on B.Cu, net +3.3V
- added copper zone on F.Cu, net +3.3V
- added copper zone on F.Cu, net +5V
Other:
- board text added: "Angle Sensor"
- board text added: "Angle Sensor NARAE, INHA Univ. 2025"
- board text added: "DIO CLK NRST TX"
- board text added: "I2C"

Commit message: fix : silkscreen
Other:
- board text added: "3.3V DIO CLK NRST TX GND"
- board text removed: "DIO CLK NRST TX"
Changed lines of the file:
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@@
 		)
 	)
-	(gr_text "DIO CLK NRST TX"
-		(at 30.5 60.25 270)
+	(gr_text "3.3V DIO CLK NRST TX GND\n"
+		(at 30.5 63 270)
 		(layer "B.SilkS")
 		(effects

Commit message: fix:readme
Parts:
- J1: value SM06B-GHS-TBT -> pinheader 2.54 6P
- moved U2 135.3 mm to (148.3, 116.9)
- moved C1 135.3 mm to (146.0, 97.2)
- moved C2 135.3 mm to (146.0, 98.8)
- moved C3 135.3 mm to (152.0, 98.5)
- moved C4 135.3 mm to (146.2, 111.2)
- moved C5 135.3 mm to (146.2, 109.8)
- moved C6 135.3 mm to (146.2, 108.2)
- moved C7 135.3 mm to (152.6, 116.4)
- moved C8 135.3 mm to (147.3, 113.9)
- moved C9 135.3 mm to (151.2, 101.5)
- moved H1 135.3 mm to (150.0, 86.9)
- moved H2 135.3 mm to (145.2, 75.5)
- moved H3 135.3 mm to (154.8, 75.5)
- moved H4 135.3 mm to (154.8, 124.5)
- moved J1 135.3 mm to (155.7, 118.7)
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