File: AeroAngleSense/AeroAngleSense.kicad_sch (KiCad schematic)
At the start: 20 parts, among them IC1 STM32F042F6P6, IC2 TMP127EDBVRQ1, IC3 TPS62842DGRR, J1 SM06B-GHS-TBT, J7 SM04B-GHS-TBT

Commit message: pcb layout done.
Parts:
- added H2, H3, H4: MountingHole, MountingHole:MountingHole_2.2mm_M2_Pad, symbol Mechanical:MountingHole
- J1: footprint Connector_PinHeader_2.54mm:PinHeader_1x01_P2.54mm_Vertical -> Connector_PinHeader_2.54mm:PinHeader_1x06_P2.54mm_Vertical
Connections:
- net at H1.2 (WIPER_): now also R2.1
- net at H1.A2 (WIPER): no longer R2.1
Other:
- moved on the sheet: C3, R2

Commit message: fix : route
Parts:
- renumbered J7 to J2, R4 to R3, R3 to R4, IC1 to U1, IC3 to U2, IC2 to U3
Changed lines of the file:
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@@
 		(on_board yes)
 		(dnp no)
-		(property "Reference" "R4"
+		(property "Reference" "R3"
 			(at 170.18 90.424 90)
 			(effects
@@
 			(project "AeroAngleSense"
 				(path "/3f9ad614-fe87-462a-b850-389279aa35f7"
-					(reference "R4")
+					(reference "R3")
 					(unit 1)
 				)
@@
 		(on_board yes)
 		(dnp no)
-		(property "Reference" "#PWR017"
+		(property "Reference" "#PWR010"
 			(at 102.87 132.08 0)
 			(effects
@@
 			(project "AeroAngleSense"
 				(path "/3f9ad614-fe87-462a-b850-389279aa35f7"
-					(reference "#PWR017")
+					(reference "#PWR010")
 					(unit 1)
 				)
@@
 		(dnp no)
 		(fields_autoplaced yes)
-		(property "Reference" "IC1"
+		(property "Reference" "U1"
 			(at 99.06 43.18 0)
 			(effects
@@
 			(project ""
 				(path "/3f9ad614-fe87-462a-b850-389279aa35f7"
-					(reference "IC1")
+					(reference "U1")
 					(unit 1)
 				)
@@
 		(dnp no)
 		(fields_autoplaced yes)
-		(property "Reference" "#PWR097"
+		(property "Reference" "#PWR013"
 			(at 144.78 138.43 0)
 			(effects
@@
 			(project "AeroAngleSense"
 				(path "/3f9ad614-fe87-462a-b850-389279aa35f7"
-					(reference "#PWR097")
+					(reference "#PWR013")
 					(unit 1)
 				)
@@
 		(dnp no)
 		(fields_autoplaced yes)
-		(property "Reference" "#PWR03"
+		(property "Reference" "#PWR06"
 			(at 54.61 50.8 0)
 			(effects
@@
 			(project ""
 				(path "/3f9ad614-fe87-462a-b850-389279aa35f7"
-					(reference "#PWR03")
+					(reference "#PWR06")
 					(unit 1)
 				)
@@
 		(dnp no)
 		(fields_autoplaced yes)
-		(property "Reference" "#PWR01"
+		(property "Reference" "#PWR03"
 			(at 20.32 66.04 0)
 			(effects
@@
 			(project "AeroAngleSense"
 				(path "/3f9ad614-fe87-462a-b850-389279aa35f7"
-					(reference "#PWR01")
+					(reference "#PWR03")
 					(unit 1)
 				)
@@
 		(dnp no)
 		(fields_autoplaced yes)
-		(property "Reference" "#PWR018"
+		(property "Reference" "#PWR011"
 			(at 102.87 149.86 0)
 			(effects
@@
 			(project "AeroAngleSense"
 				(path "/3f9ad614-fe87-462a-b850-389279aa35f7"
-					(reference "#PWR018")
+					(reference "#PWR011")
 					(unit 1)
 				)
@@
 		(on_board yes)
 		(dnp no)
-		(property "Reference" "R3"
+		(property "Reference" "R4"
 			(at 209.55 69.85 90)
 			(effects
@@
 			(project ""
 				(path "/3f9ad614-fe87-462a-b850-389279aa35f7"
-					(reference "R3")
+					(reference "R4")
 					(unit 1)
 				)
@@
 		(dnp no)
 		(fields_autoplaced yes)
-		(property "Reference" "#PWR04"
+		(property "Reference" "#PWR08"
 			(at 81.28 97.79 0)
 			(effects
@@
 			(project "AeroAngleSense"
 				(path "/3f9ad614-fe87-462a-b850-389279aa35f7"
-					(reference "#PWR04")
+					(reference "#PWR08")
 					(unit 1)
 				)
@@
 		(on_board yes)
 		(dnp no)
-		(property "Reference" "#PWR096"
+		(property "Reference" "#PWR012"
 			(at 138.43 132.08 0)
 			(effects
@@
 			(project "AeroAngleSense"
 				(path "/3f9ad614-fe87-462a-b850-389279aa35f7"
-					(reference "#PWR096")
+					(reference "#PWR012")
 					(unit 1)
 				)
@@
 		(dnp no)
 		(fields_autoplaced yes)
-		(property "Reference" "#PWR09"
+		(property "Reference" "#PWR016"
 			(at 168.91 62.23 0)
 			(effects
@@
 			(project ""
 				(path "/3f9ad614-fe87-462a-b850-389279aa35f7"
-					(reference "#PWR09")
+					(reference "#PWR016")
 					(unit 1)
 				)
@@
 		(dnp no)
 		(fields_autoplaced yes)
-		(property "Reference" "#PWR020"
+		(property "Reference" "#PWR02"
 			(at 30.48 62.23 0)
 			(effects
@@
 			(project "AeroAngleSense"
 				(path "/3f9ad614-fe87-462a-b850-389279aa35f7"
-					(reference "#PWR020")
+					(reference "#PWR02")
 					(unit 1)
 				)
@@
 		(dnp no)
 		(fields_autoplaced yes)
-		(property "Reference" "#PWR015"
+		(property "Reference" "#PWR022"
 			(at 220.98 91.44 0)
 			(effects
@@
 			(project ""
 				(path "/3f9ad614-fe87-462a-b850-389279aa35f7"
-					(reference "#PWR015")
+					(reference "#PWR022")
 					(unit 1)
 				)
@@
 		(dnp no)
 		(fields_autoplaced yes)
-		(property "Reference" "IC2"
+		(property "Reference" "U3"
 			(at 189.23 81.28 0)
 			(effects
@@
 			(project ""
 				(path "/3f9ad614-fe87-462a-b850-389279aa35f7"
-					(reference "IC2")
+					(reference "U3")
 					(unit 1)
 				)
@@
 		(dnp no)
 		(fields_autoplaced yes)
-		(property "Reference" "#PWR019"
+		(property "Reference" "#PWR01"
 			(at 30.48 59.69 0)
 			(effects
@@
 			(project "AeroAngleSense"
 				(path "/3f9ad614-fe87-462a-b850-389279aa35f7"
-					(reference "#PWR019")
+					(reference "#PWR01")
 					(unit 1)
 				)
@@
 		(dnp no)
 		(fields_autoplaced yes)
-		(property "Reference" "#PWR012"
+		(property "Reference" "#PWR019"
 			(at 201.93 77.47 0)
 			(effects
@@
 			(project "AeroAngleSense"
 				(path "/3f9ad614-fe87-462a-b850-389279aa35f7"
-					(reference "#PWR012")
+					(reference "#PWR019")
 					(unit 1)
 				)
@@
 		(dnp no)
 		(fields_autoplaced yes)
-		(property "Reference" "#PWR08"
+		(property "Reference" "#PWR015"
 			(at 157.48 68.58 0)
 			(effects
@@
 			(project ""
 				(path "/3f9ad614-fe87-462a-b850-389279aa35f7"
-					(reference "#PWR08")
+					(reference "#PWR015")
 					(unit 1)
 				)
@@
 		(on_board yes)
 		(dnp no)
-		(property "Reference" "J7"
+		(property "Reference" "J2"
 			(at 130.81 128.016 0)
 			(effects
@@
 			(project "AeroAngleSense"
 				(path "/3f9ad614-fe87-462a-b850-389279aa35f7"
-					(reference "J7")
+					(reference "J2")
 					(unit 1)
 				)
@@
 		(dnp no)
 		(fields_autoplaced yes)
-		(property "Reference" "#PWR06"
+		(property "Reference" "#PWR07"
 			(at 74.93 111.76 0)
 			(effects
@@
 			(project "AeroAngleSense"
 				(path "/3f9ad614-fe87-462a-b850-389279aa35f7"
-					(reference "#PWR06")
+					(reference "#PWR07")
 					(unit 1)
 				)
@@
 		(dnp no)
 		(fields_autoplaced yes)
-		(property "Reference" "#PWR016"
+		(property "Reference" "#PWR023"
 			(at 220.98 104.14 0)
 			(effects
@@
 			(project ""
 				(path "/3f9ad614-fe87-462a-b850-389279aa35f7"
-					(reference "#PWR016")
+					(reference "#PWR023")
 					(unit 1)
 				)
@@
 		(dnp no)
 		(fields_autoplaced yes)
-		(property "Reference" "#PWR02"
+		(property "Reference" "#PWR05"
 			(at 48.26 63.5 0)
 			(effects
@@
 			(project ""
 				(path "/3f9ad614-fe87-462a-b850-389279aa35f7"
-					(reference "#PWR02")
+					(reference "#PWR05")
 					(unit 1)
 				)
@@
 		(dnp no)
 		(fields_autoplaced yes)
-		(property "Reference" "#PWR021"
+		(property "Reference" "#PWR04"
 			(at 40.64 68.58 0)
 			(effects
@@
 			(project "AeroAngleSense"
 				(path "/3f9ad614-fe87-462a-b850-389279aa35f7"
-					(reference "#PWR021")
+					(reference "#PWR04")
 					(unit 1)
 				)
@@
 		(dnp no)
 		(fields_autoplaced yes)
-		(property "Reference" "#PWR07"
+		(property "Reference" "#PWR014"
 			(at 149.86 63.5 0)
 			(effects
@@
 			(project ""
 				(path "/3f9ad614-fe87-462a-b850-389279aa35f7"
-					(reference "#PWR07")
+					(reference "#PWR014")
 					(unit 1)
 				)
@@
 		(dnp no)
 		(fields_autoplaced yes)
-		(property "Reference" "#PWR011"
+		(property "Reference" "#PWR018"
 			(at 176.53 74.93 0)
 			(effects
@@
 			(project ""
 				(path "/3f9ad614-fe87-462a-b850-389279aa35f7"
-					(reference "#PWR011")
+					(reference "#PWR018")
 					(unit 1)
 				)
@@
 		(dnp no)
 		(fields_autoplaced yes)
-		(property "Reference" "#PWR014"
+		(property "Reference" "#PWR021"
 			(at 213.36 74.93 0)
 			(effects
@@
 			(project ""
 				(path "/3f9ad614-fe87-462a-b850-389279aa35f7"
-					(reference "#PWR014")
+					(reference "#PWR021")
 					(unit 1)
 				)
@@
 		(dnp no)
 		(fields_autoplaced yes)
-		(property "Reference" "#PWR010"
+		(property "Reference" "#PWR017"
 			(at 168.91 74.93 0)
 			(effects
@@
 			(project ""
 				(path "/3f9ad614-fe87-462a-b850-389279aa35f7"
-					(reference "#PWR010")
+					(reference "#PWR017")
 					(unit 1)
 				)
@@
 		(dnp no)
 		(fields_autoplaced yes)
-		(property "Reference" "#PWR05"
+		(property "Reference" "#PWR09"
 			(at 81.28 107.95 0)
 			(effects
@@
 			(project "AeroAngleSense"
 				(path "/3f9ad614-fe87-462a-b850-389279aa35f7"
-					(reference "#PWR05")
+					(reference "#PWR09")
 					(unit 1)
 				)
@@
 		(dnp no)
 		(fields_autoplaced yes)
-		(property "Reference" "#PWR013"
+		(property "Reference" "#PWR020"
 			(at 213.36 62.23 0)
 			(effects
@@
 			(project ""
 				(path "/3f9ad614-fe87-462a-b850-389279aa35f7"
-					(reference "#PWR013")
+					(reference "#PWR020")
 					(unit 1)
 				)
@@
 		(on_board yes)
 		(dnp no)
-		(property "Reference" "IC3"
+		(property "Reference" "U2"
 			(at 189.23 54.102 0)
 			(effects
@@
 			(project ""
 				(path "/3f9ad614-fe87-462a-b850-389279aa35f7"
-					(reference "IC3")
+					(reference "U2")
 					(unit 1)
 				)

Commit message: fix:readme
Parts:
- J1: value SM06B-GHS-TBT -> pinheader 2.54 6P; LCSC C133065 -> (none)
Other:
- note added: "DC to DC Buck"
- note added: "Hole"
- note added: "I2C"
- note added: "I2C_SCL : PA9 I2C_SDA : PA10"
- note added: "M2"
- note added: "MCU"
- note added: "POT_SEN : PB1"
- note added: "Potentiometer"
- note added: "SWDIO : PA13 SWCLK : PA14 NRST : NRST(14) USART2_TX : PA2"
- note added: "TMP_SCLK : PA5 TMP_MOSI : PA7 TMP_MISO : PA6"
- note added: "Temperature Sensor"
- company: (none) -> NARAE
- title: (none) -> AeroAngleSense
- moved on the sheet: C1, C2, C3, C4, C5, C6, C7, C8, C9, H1, H2, H3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
